File: Hardware/KiCad/Power-Management/Power-Management.kicad_pcb (KiCad board)
At the start: 2 copper layers, 108 x 67 mm, 51 parts, among them IC1 RT9080-33GJ5, J1 Screw_Terminal_01x02, J2 Conn_01x06, J3 Screw_Terminal_01x02, K1 FINDER-36.11, Q1 BC817, T1 ZMPT101B, U1 STM32F401CCU6, U2 ACS758xCB-050B-PFF, U3 ESP-01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

Commit message: project libraries
Parts:
- removed F1: Fuse, Fuse:Fuseholder_Clip-5x20mm_Keystone_3512P_Inline_P23.62x7.27mm_D1.02x2.41x1.02x1.57mm_Horizontal
