File: Hardware/KiCad/Power-Management/Power-Management.kicad_pcb (KiCad board)
At the start: 2 copper layers, 108 x 67 mm, 50 parts, among them IC1 RT9080-33GJ5, J1 Screw_Terminal_01x02, J2 Conn_01x06, J3 Screw_Terminal_01x02, K1 FINDER-36.11, Q1 BC817, T1 ZMPT101B, U1 STM32F401CCU6, U2 ACS758xCB-050B-PFF, U3 ESP-01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

Commit message: feat: hierarchical sheet
Parts:
- removed U5: LM358ADE4, LM358ADE4:SOIC127P599X175-8N
- added R14: 10K, Resistor_SMD:R_0805_2012Metric_Pad1.20x1.40mm_HandSolder, F.Cu at (168.4, 95.6)
- added U4: LM358ADE4, LM358ADE4:SOIC127P599X175-8N, F.Cu at (174.7, 86.3)
- C11: value 1uF -> 1nF
- C12: value 1nF -> 1uF
- R10, R6: value 100K -> 10K
- R12: value 10K -> 1K
- R7, R9: value 10K -> 100K
- moved R7 13.9 mm to (174.5, 80.3)
- moved R9 8.55 mm to (174.2, 91.1)
- moved R6 8.47 mm to (181.8, 84.6), turned to -90 degrees
- moved R3 6.25 mm to (163.0, 81.5), turned to 90 degrees
- moved R5 6.23 mm to (167.7, 85.7), turned to 180 degrees
- moved J3 5.76 mm to (128.5, 98.9), turned to -90 degrees
- moved C12 4.00 mm to (172.2, 91.1)
- moved C11 3.99 mm to (176.1, 91.1)
- moved R12 3.30 mm to (171.9, 96.6)
- moved R10 3.15 mm to (173.2, 94.1), turned to 180 degrees
- moved R8 2.00 mm to (179.8, 84.6)
- moved J1 1.50 mm to (128.5, 93.2)
- moved C7 1.16 mm to (190.2, 62.2)
- moved K1 0.85 mm to (151.1, 98.0)
- moved VR1 0.41 mm to (164.9, 90.7)
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Connections:
- C10 pad 1: Net-(U5-2IN-) -> Net-(U4-2IN-)
- C10 pad 2: Net-(U5-2OUT) -> Net-(U4-2OUT)
- C11 pad 1: Net-(C11-Pad1) -> Net-(U4-1IN-)
- C11 pad 2: Net-(C11-Pad2) -> PIN_ZMPT101B
- C12 pad 1: Net-(U5-1IN-) -> Net-(C12-Pad1)
- C12 pad 2: PIN_ZMPT101B -> Net-(C12-Pad2)
- R10 pad 1: PIN_ZMPT101B -> Net-(U4-1IN-)
- R10 pad 2: Net-(U5-1IN-) -> Net-(C12-Pad1)
- R2 pad 1: Net-(U5-2IN+) -> Net-(U4-2IN+)
- R3 pad 1: Net-(U5-2IN-) -> Net-(U4-2IN+)
- R3 pad 2: Net-(C9-Pad2) -> +5V
- R4 pad 1: Net-(U5-2IN+) -> Net-(U4-2IN+)
- R5 pad 1: Net-(U5-2IN+) -> Net-(U4-2IN-)
- R5 pad 2: +5V -> Net-(C9-Pad2)
- R6 pad 1: Net-(U5-2OUT) -> GND
- R6 pad 2: Net-(U5-2IN-) -> Net-(U4-1IN+)
- R7 pad 1: Net-(U5-1IN-) -> Net-(U4-2OUT)
- R7 pad 2: Net-(C11-Pad1) -> Net-(U4-2IN-)
- R8 pad 1: GND -> +5V
- R8 pad 2: Net-(U5-1IN+) -> Net-(U4-1IN+)
- R9 pad 1: +5V -> PIN_ZMPT101B
- R9 pad 2: Net-(U5-1IN+) -> Net-(U4-1IN-)
- T1 pad 4: Net-(U5-2IN+) -> Net-(U4-2IN+)
- VR1 pad 1: Net-(U5-2OUT) -> Net-(U4-2OUT)
- VR1 pad 2: Net-(C11-Pad2) -> Net-(C12-Pad2)
Routing:
- net Net-(U5-2IN+): track 26.6 -> 0.00 mm, vias 2 -> 0
- net Net-(U4-2IN+): track 0.00 -> 26.5 mm, vias 0 -> 2
- net Net-(U5-2OUT): track 17.7 -> 0.00 mm
- net Net-(U4-2OUT): track 0.00 -> 17.2 mm
- net Net-(U5-1IN-): track 13.9 -> 0.00 mm
- net Net-(U4-1IN-): track 0.00 -> 13.9 mm
- net Net-(U4-2IN-): track 0.00 -> 12.4 mm
- net Net-(U5-2IN-): track 12.4 -> 0.00 mm
- net Net-(C12-Pad2): track 0.00 -> 10.9 mm
- net Net-(C11-Pad2): track 10.4 -> 0.00 mm
- net Net-(U5-1IN+): track 4.59 -> 0.00 mm
- net Net-(U4-1IN+): track 0.00 -> 4.59 mm
- net PIN_RELAY: track 52.9 -> 48.9 mm
- net F/N-1 Borne: track 16.4 -> 12.9 mm
- net Net-(Q1-B): track 2.98 -> 6.32 mm
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