File: Hardware/KiCad/Power-Management/Power-Management.kicad_sch (KiCad schematic)
At the start: 31 parts, among them IC1 RT9080-33GJ5, J1 Screw_Terminal_01x02, J2 Conn_01x06, J3 Screw_Terminal_01x02, K1 FINDER-36.11, Q1 BC817, U1 STM32F401CCU6, U3 ESP-01, Y1 25Mhz

Commit message: troca de sensor de corrente
Parts:
- removed C16, C6: 100nF, Capacitor_SMD:C_0805_2012Metric, symbol Device:C
- removed C2, C7: 10pF, Capacitor_SMD:C_0805_2012Metric, symbol Device:C
- removed C5: 22uF 10V, Capacitor_SMD:C_0805_2012Metric, symbol Device:C
- removed U1: STM32F401CCU6, Package_DFN_QFN:QFN-48-1EP_7x7mm_P0.5mm_EP3.5x3.5mm, symbol MCU_ST_STM32F4:STM32F401CCUx
- removed Y1: 25Mhz, TSX-3225_25.0000MF10Z-W:XTAL_TSX-3225_25.0000MF10Z-W, symbol TSX-3225_25.0000MF10Z-W:TSX-3225_25.0000MF10Z-W
- added C17, C18, C20, C21, C22: 100nF, Capacitor_SMD:C_0805_2012Metric, symbol Device:C
- added C19: 10uF, Capacitor_SMD:C_0805_2012Metric, symbol Device:C
- added C23, C24: 10pF, Capacitor_SMD:C_0805_2012Metric, symbol Device:C
- added R15: 10K, Resistor_SMD:R_0805_2012Metric_Pad1.20x1.40mm_HandSolder, symbol Device:R
- added S1: SKRKAEE010, SKRKAEE010:SKRK, symbol SKRKAEE010:SKRKAEE010
- added U5: STM32F103C8Tx, Package_QFP:LQFP-48_7x7mm_P0.5mm, symbol MCU_ST_STM32F1:STM32F103C8Tx
- added Y2: 16Mhz, TSX-3225_25.0000MF10Z-W:XTAL_TSX-3225_25.0000MF10Z-W, symbol TSX-3225_25.0000MF10Z-W:TSX-3225_25.0000MF10Z-W
- C1: value 5pF -> 100nF
Connections:
- net +3V3: now also C17.2, C18.2, C19.2, C20.2, C21.2, R15.1, U5.1 (VBAT), U5.24 (VDD), U5.36 (VDD), U5.48 (VDD), U5.9 (VDDA)
- net F/N-1 Borne: no longer K1.14
- net F/N-2: now also K1.12
- net GND: now also C17.1, C18.1, C19.1, C20.1, C21.1, C22.1, C23.1, C24.1, S1.1, U5.23 (VSS), U5.35 (VSS), U5.47 (VSS), U5.8 (VSSA), Y2.2 (GND), Y2.4 (GND)
- net PIN_ACS758: now also U5.11 (PA1)
- net PIN_LED_RGB: now also U5.40 (PB4)
- net PIN_RELAY: now also U5.20 (PB2)
- net PIN_ZMPT101B: now also U5.12 (PA2)
- net RXD1: now also U5.31 (PA10)
- net SWCLK: now also U5.37 (PA14)
- net SWDIO: now also U5.34 (PA13)
- net TXD1: now also U5.30 (PA9)
- net CONFIG_WIFI: now reaches C1.2
- net CONFIG_WIFI: now also R11.2, S2.2, U5.39 (PB3)
- net F/N-1 | ACS58 renamed F/N-1 HOLE
- net RXD6 renamed RXD3
- net RXD3: now also U5.22 (PB11)
- net TXD6 renamed TXD3
- net TXD3: now also U5.21 (PB10)
- new net: C22.2, R15.2, S1.2, U5.7 (NRST)
- new net: C23.2, U5.5 (PD0), Y2.1
- new net: C24.2, U5.6 (PD1), Y2.3
- no-connect marks 37 -> 10
Other:
- note added: "HSE_IN"
- note added: "HSE_OUT"
- moved on the sheet: C8, D1, J2
